File: Hardware/EPS/Mounting_Holes.kicad_sch (KiCad schematic)
At the start: 4 parts, among them M3 MountingHole_Pad

Commit message: Fuse, Power Switch to 3.3V, connector ESD Prot.
v0.0.2
Other:
- title: (none) -> EPS Schematics
Changed lines of the file:
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@@
 (kicad_sch (version 20211123) (generator eeschema)
   (paper "A4")
+  (title_block
+    (title "EPS Schematics")
+    (date "2023-04-08")
+    (rev "v0.0.2")
+    (comment 1 "e-mail: carmamo.95@gmail.com")
+    (comment 2 "Author: Carlos Martinez Mora")
+  )
   (junction (at 152.4 92.71) (diameter 0) (color 0 0 0 0)
   )

Commit message: MPPT IC Routing & layout
Parts:
- M1201, M1202, M1203, M1204: renamed from M3; footprint (none) -> MountingHole:MountingHole_3.2mm_M3_ISO7380_Pad
Changed lines of the file:
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@@
   (symbol (lib_id "Mechanical:MountingHole_Pad") (at 142.24 92.71 90) (unit 1)
     (in_bom yes) (on_board yes) (fields_autoplaced)
-    (property "Reference" "M3" (id 0) (at 140.97 87.2322 90))
+    (property "Reference" "M1203" (id 0) (at 140.97 87.2322 90))
     (property "Value" "MountingHole_Pad" (id 1) (at 140.97 89.7691 90))
-    (property "Footprint" "" (id 2) (at 142.24 92.71 0)
+    (property "Footprint" "MountingHole:MountingHole_3.2mm_M3_ISO7380_Pad" (id 2) (at 142.24 92.71 0)
       (effects (font (size 1.27 1.27)) hide)
     )
@@
   (symbol (lib_id "Mechanical:MountingHole_Pad") (at 142.24 83.82 90) (unit 1)
     (in_bom yes) (on_board yes) (fields_autoplaced)
-    (property "Reference" "M3" (id 0) (at 140.97 78.3422 90))
+    (property "Reference" "M1202" (id 0) (at 140.97 78.3422 90))
     (property "Value" "MountingHole_Pad" (id 1) (at 140.97 80.8791 90))
-    (property "Footprint" "" (id 2) (at 142.24 83.82 0)
+    (property "Footprint" "MountingHole:MountingHole_3.2mm_M3_ISO7380_Pad" (id 2) (at 142.24 83.82 0)
       (effects (font (size 1.27 1.27)) hide)
     )
@@
   (symbol (lib_id "power:GND") (at 152.4 101.6 0) (unit 1)
     (in_bom yes) (on_board yes) (fields_autoplaced)
-    (property "Reference" "#PWR?" (id 0) (at 152.4 107.95 0)
+    (property "Reference" "#PWR01201" (id 0) (at 152.4 107.95 0)
       (effects (font (size 1.27 1.27)) hide)
     )
@@
   (symbol (lib_id "Mechanical:MountingHole_Pad") (at 142.24 74.93 90) (unit 1)
     (in_bom yes) (on_board yes) (fields_autoplaced)
-    (property "Reference" "M3" (id 0) (at 140.97 69.4522 90))
+    (property "Reference" "M1201" (id 0) (at 140.97 69.4522 90))
     (property "Value" "MountingHole_Pad" (id 1) (at 140.97 71.9891 90))
-    (property "Footprint" "" (id 2) (at 142.24 74.93 0)
+    (property "Footprint" "MountingHole:MountingHole_3.2mm_M3_ISO7380_Pad" (id 2) (at 142.24 74.93 0)
       (effects (font (size 1.27 1.27)) hide)
     )
@@
   (symbol (lib_id "Mechanical:MountingHole_Pad") (at 142.24 101.6 90) (unit 1)
     (in_bom yes) (on_board yes) (fields_autoplaced)
-    (property "Reference" "M3" (id 0) (at 140.97 96.1222 90))
+    (property "Reference" "M1204" (id 0) (at 140.97 96.1222 90))
     (property "Value" "MountingHole_Pad" (id 1) (at 140.97 98.6591 90))
-    (property "Footprint" "" (id 2) (at 142.24 101.6 0)
+    (property "Footprint" "MountingHole:MountingHole_3.2mm_M3_ISO7380_Pad" (id 2) (at 142.24 101.6 0)
       (effects (font (size 1.27 1.27)) hide)
     )

Commit message: Finished EPS - v0.1.0
Parts:
- M1201, M1202, M1203, M1204: footprint MountingHole:MountingHole_3.2mm_M3_ISO7380_Pad -> MountingHole:MountingHole_3.2mm_M3_Pad_Via
Changed lines of the file:
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@@
   (title_block
     (title "EPS Schematics")
-    (date "2023-04-08")
-    (rev "v0.0.3")
-    (comment 1 "e-mail: ")
+    (date "2023-04-19")
+    (rev "v0.1.0")
+    (comment 1 "LinkedIn: linkedin.com/in/carlos-martinez-mora-7b2023230/")
     (comment 2 "Author: Carlos Martinez Mora")
   )
@@
     (property "Reference" "M1203" (id 0) (at 140.97 87.2322 90))
     (property "Value" "MountingHole_Pad" (id 1) (at 140.97 89.7691 90))
-    (property "Footprint" "MountingHole:MountingHole_3.2mm_M3_ISO7380_Pad" (id 2) (at 142.24 92.71 0)
+    (property "Footprint" "MountingHole:MountingHole_3.2mm_M3_Pad_Via" (id 2) (at 142.24 92.71 0)
       (effects (font (size 1.27 1.27)) hide)
     )
@@
     (property "Reference" "M1202" (id 0) (at 140.97 78.3422 90))
     (property "Value" "MountingHole_Pad" (id 1) (at 140.97 80.8791 90))
-    (property "Footprint" "MountingHole:MountingHole_3.2mm_M3_ISO7380_Pad" (id 2) (at 142.24 83.82 0)
+    (property "Footprint" "MountingHole:MountingHole_3.2mm_M3_Pad_Via" (id 2) (at 142.24 83.82 0)
       (effects (font (size 1.27 1.27)) hide)
     )
@@
     (property "Reference" "M1201" (id 0) (at 140.97 69.4522 90))
     (property "Value" "MountingHole_Pad" (id 1) (at 140.97 71.9891 90))
-    (property "Footprint" "MountingHole:MountingHole_3.2mm_M3_ISO7380_Pad" (id 2) (at 142.24 74.93 0)
+    (property "Footprint" "MountingHole:MountingHole_3.2mm_M3_Pad_Via" (id 2) (at 142.24 74.93 0)
       (effects (font (size 1.27 1.27)) hide)
     )
@@
     (property "Reference" "M1204" (id 0) (at 140.97 96.1222 90))
     (property "Value" "MountingHole_Pad" (id 1) (at 140.97 98.6591 90))
-    (property "Footprint" "MountingHole:MountingHole_3.2mm_M3_ISO7380_Pad" (id 2) (at 142.24 101.6 0)
+    (property "Footprint" "MountingHole:MountingHole_3.2mm_M3_Pad_Via" (id 2) (at 142.24 101.6 0)
       (effects (font (size 1.27 1.27)) hide)
     )
