File: Hardware/PAYLOAD/Power.kicad_sch (KiCad schematic)
At the start: 0 parts

Commit message: Updated to KiCAD 7.0
Parts:
- added U?: LT1930ES5#TRMPBF, LT1930ES5#TRMPBF:SOT95P280X145-5N, symbol LT1930ES5#TRMPBF:LT1930ES5#TRMPBF
Changed lines of the file:
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@@
 (kicad_sch (version 20211123) (generator eeschema)
   (paper "A4")
+  (symbol (lib_id "LT1930ES5#TRMPBF:LT1930ES5#TRMPBF") (at 124.46 85.09 0) (unit 1)
+    (in_bom yes) (on_board yes) (fields_autoplaced)
+    (property "Reference" "U?" (id 0) (at 138.43 73.7764 0))
+    (property "Value" "LT1930ES5#TRMPBF" (id 1) (at 138.43 76.3133 0))
+    (property "Footprint" "LT1930ES5#TRMPBF:SOT95P280X145-5N" (id 2) (at 124.46 85.09 0)
+      (effects (font (size 1.27 1.27)) hide)
+    )
+    (property "Datasheet" "" (id 3) (at 124.46 85.09 0)
+      (effects (font (size 1.27 1.27)) hide)
+    )
+    (property "Reference_1" "IC" (id 4) (at 138.43 78.8502 0))
+    (property "Value_1" "LT1930ES5#TRMPBF" (id 5) (at 138.43 81.3871 0))
+    (property "Footprint_1" "SOT95P280X145-5N" (id 6) (at 148.59 180.01 0)
+      (effects (font (size 1.27 1.27)) (justify left top) hide)
+    )
+    (property "Datasheet_1" "https://datasheet.datasheetarchive.com/originals/distributors/SFDatasheet-4/sf-00091027.pdf" (id 7) (at 148.59 280.01 0)
+      (effects (font (size 1.27 1.27)) (justify left top) hide)
+    )
+    (property "Height" "1.45" (id 8) (at 148.59 480.01 0)
+      (effects (font (size 1.27 1.27)) (justify left top) hide)
+    )
+    (property "Manufacturer_Name" "Analog Devices" (id 9) (at 148.59 580.01 0)
+      (effects (font (size 1.27 1.27)) (justify left top) hide)
+    )
+    (property "Manufacturer_Part_Number" "LT1930ES5#TRMPBF" (id 10) (at 148.59 680.01 0)
+      (effects (font (size 1.27 1.27)) (justify left top) hide)
+    )
+    (property "Mouser Part Number" "584-LT1930ES5#TRMPBF" (id 11) (at 148.59 780.01 0)
+      (effects (font (size 1.27 1.27)) (justify left top) hide)
+    )
+    (property "Mouser Price/Stock" "https://www.mouser.co.uk/ProductDetail/Analog-Devices/LT1930ES5TRMPBF?qs=ytflclh7QUXsZW533VXHKw%3D%3D" (id 12) (at 148.59 880.01 0)
+      (effects (font (size 1.27 1.27)) (justify left top) hide)
+    )
+    (property "Arrow Part Number" "LT1930ES5#TRMPBF" (id 13) (at 148.59 980.01 0)
+      (effects (font (size 1.27 1.27)) (justify left top) hide)
+    )
+    (property "Arrow Price/Stock" "https://www.arrow.com/en/products/lt1930es5trmpbf/analog-devices?region=nac" (id 14) (at 148.59 1080.01 0)
+      (effects (font (size 1.27 1.27)) (justify left top) hide)
+    )
+    (pin "1")
+    (pin "2")
+    (pin "3")
+    (pin "4")
+    (pin "5")
+  )
 )
